Commit message: turned encoder into a simple python class

File: src/hadabot_description/src/description/hadabot_description.urdf (robot description, URDF)
Before this commit: robot hadabot, 3 links, 2 joints
Links:
- link base_link: geometry collision box size=${base_length} ${base_width} ${base_height}; visual box size=${base_length} ${base_width} ${base_height}
- link front_caster: geometry collision sphere radius=${(wheel_radius+wheel_zoff-(base_height/2))}; visual sphere radius=${(wheel_radius)}
Joints:
- joint caster_joint: origin xyz=${caster_xoff} 0.0 ${-(base_height/2)} rpy=0 0 0 -> xyz=${caster_xoff} 0.0 ${-(base_height)} rpy=0 0 0

Commit message: added robot state publisher and URDF

File: src/hadabot_description/src/description/hadabot_description.urdf (robot description, URDF)
Before this commit: robot hadabot, 3 links, 2 joints
Links:
- added link laser; visual cylinder length=0.051 radius=0.0225
Joints:
- added joint lidar_joint: type fixed, parent base_link, child laser, origin xyz=0.0 0 0.20 rpy=0 0 0
